Commit message: fix: refactoring the pybullet_collision_test.py into smaller helper functions places in the correct theme file

File: duckify_simulation/urdf/ur3e.urdf (robot description, URDF)
Before this commit: robot ur3e, 16 links, 15 joints
Joints:
- joint pen_joint: origin xyz=0 0 0.101 rpy=3.141592653589793 0 0 -> xyz=0 0 0.1091 rpy=3.141592653589793 0 0

Commit message: feat: adding 6 angles plot (matplotlib)

File: duckify_simulation/urdf/ur3e.urdf (robot description, URDF)
Before this commit: robot ur3e, 16 links, 15 joints
Joints:
- joint pen_joint: origin xyz=0 0 0.1091 rpy=3.141592653589793 0 0 -> xyz=0 0 0.1051 rpy=3.141592653589793 0 0
